File: rooDialino-KiCad/roodialino.sch (KiCad schematic (older format))
At the start: 58 parts, among them J1 Raspi Connector, J2 ICSP, J3 FTDI, J4 IR Receiver, J5 IR LED, Q1 2N7002, Q2 2N7002, Q3 2N7002, SW1 SW_Push, U1 ATmega328P, U2 TSOP312xx, U3 TXS0108EPW, Y1 16MHz

Commit message: Looking good, that PCB
Parts:
- removed TP1: D9, TestPoint:TestPoint_THTPad_D1.5mm_Drill0.7mm, symbol Connector:TestPoint
- removed TP2: A0, TestPoint:TestPoint_THTPad_D1.5mm_Drill0.7mm, symbol Connector:TestPoint
- removed TP3: GPIO5, TestPoint:TestPoint_THTPad_D1.5mm_Drill0.7mm, symbol Connector:TestPoint
- removed TP4: GPIO6, TestPoint:TestPoint_THTPad_D1.5mm_Drill0.7mm, symbol Connector:TestPoint
- removed TP5: IRTX, TestPoint:TestPoint_THTPad_D1.5mm_Drill0.7mm, symbol Connector:TestPoint
- removed TP6: IRRCV, TestPoint:TestPoint_THTPad_D1.5mm_Drill0.7mm, symbol Connector:TestPoint
- removed TP7: GND, TestPoint:TestPoint_THTPad_D1.5mm_Drill0.7mm, symbol Connector:TestPoint
- removed TP8: +3.3V, TestPoint:TestPoint_THTPad_D1.5mm_Drill0.7mm, symbol Connector:TestPoint
- removed TP9: +5V, TestPoint:TestPoint_THTPad_D1.5mm_Drill0.7mm, symbol Connector:TestPoint
- D7: footprint LED_THT:LED_D5.0mm_Clear -> LED_THT:LED_D5.0mm_IRBlack
Changed lines of the file:
@@
 Text Label 2150 1300 0    50   ~ 0
 LEDRSTATE
-$Comp
-L Connector:TestPoint TP1
-U 1 1 5E0E3D08
-P 9400 850
-F 0 "TP1" V 9350 1050 50  0000 L CNN
-F 1 "D9" V 9450 850 50  0000 L CNN
-F 2 "TestPoint:TestPoint_THTPad_D1.5mm_Drill0.7mm" H 9600 850 50  0001 C CNN
-F 3 "~" H 9600 850 50  0001 C CNN
-	1    9400 850
-	0    1    1    0
-$EndComp
 Text Label 2150 3000 0    50   ~ 0
 VOL+5
@@
 F 0 "D7" H 5250 1900 50  0000 R CNN
 F 1 "LED" H 5250 2000 50  0000 R CNN
-F 2 "LED_THT:LED_D5.0mm_Clear" H 5200 1800 50  0001 C CNN
+F 2 "LED_THT:LED_D5.0mm_IRBlack" H 5200 1800 50  0001 C CNN
 F 3 "~" H 5200 1800 50  0001 C CNN
 	1    5200 1800
@@
 Text Label 2150 2000 0    50   ~ 0
 A0
-$Comp
-L Connector:TestPoint TP2
-U 1 1 61B69443
-P 9400 1000
-F 0 "TP2" V 9350 1200 50  0000 L CNN
-F 1 "A0" V 9450 1000 50  0000 L CNN
-F 2 "TestPoint:TestPoint_THTPad_D1.5mm_Drill0.7mm" H 9600 1000 50  0001 C CNN
-F 3 "~" H 9600 1000 50  0001 C CNN
-	1    9400 1000
-	0    1    1    0
-$EndComp
 Text Label 1900 5150 0    50   ~ 0
 TX3
@@
 Wire Wire Line
 	1100 6350 1250 6350
-$Comp
-L Connector:TestPoint TP3
-U 1 1 61D2E239
-P 9400 1300
-F 0 "TP3" V 9350 1500 50  0000 L CNN
-F 1 "GPIO5" V 9450 1150 50  0000 L CNN
-F 2 "TestPoint:TestPoint_THTPad_D1.5mm_Drill0.7mm" H 9600 1300 50  0001 C CNN
-F 3 "~" H 9600 1300 50  0001 C CNN
-	1    9400 1300
-	0    1    1    0
-$EndComp
-$Comp
-L Connector:TestPoint TP4
-U 1 1 61D2E699
-P 9400 1450
-F 0 "TP4" V 9350 1650 50  0000 L CNN
-F 1 "GPIO6" V 9450 1300 50  0000 L CNN
-F 2 "TestPoint:TestPoint_THTPad_D1.5mm_Drill0.7mm" H 9600 1450 50  0001 C CNN
-F 3 "~" H 9600 1450 50  0001 C CNN
-	1    9400 1450
-	0    1    1    0
-$EndComp
 Wire Wire Line
 	2000 2900 2150 2900
@@
 VOL+5
 $Comp
-L Connector:TestPoint TP5
-U 1 1 61EBC057
-P 9400 2100
-F 0 "TP5" V 9350 2300 50  0000 L CNN
-F 1 "IRTX" V 9450 2000 50  0000 L CNN
-F 2 "TestPoint:TestPoint_THTPad_D1.5mm_Drill0.7mm" H 9600 2100 50  0001 C CNN
-F 3 "~" H 9600 2100 50  0001 C CNN
-	1    9400 2100
-	0    1    1    0
-$EndComp
-$Comp
-L Connector:TestPoint TP6
-U 1 1 61EBC300
-P 9400 2250
-F 0 "TP6" V 9350 2450 50  0000 L CNN
-F 1 "IRRCV" V 9450 2100 50  0000 L CNN
-F 2 "TestPoint:TestPoint_THTPad_D1.5mm_Drill0.7mm" H 9600 2250 50  0001 C CNN
-F 3 "~" H 9600 2250 50  0001 C CNN
-	1    9400 2250
-	0    1    1    0
-$EndComp
-Text Label 9400 850  2    50   ~ 0
-D9
-Text Label 9400 1000 2    50   ~ 0
-A0
-Text Label 9400 1300 2    50   ~ 0
-GPIO5
-Text Label 9400 1450 2    50   ~ 0
-GPIO6
-Text Label 9400 2100 2    50   ~ 0
-IRTX
-Text Label 9400 2250 2    50   ~ 0
-IRRCV
-$Comp
-L Connector:TestPoint TP7
-U 1 1 61EBCD0A
-P 9400 2450
-F 0 "TP7" V 9350 2650 50  0000 L CNN
-F 1 "GND" V 9450 2400 50  0000 L CNN
-F 2 "TestPoint:TestPoint_THTPad_D1.5mm_Drill0.7mm" H 9600 2450 50  0001 C CNN
-F 3 "~" H 9600 2450 50  0001 C CNN
-	1    9400 2450
-	0    1    1    0
-$EndComp
-$Comp
-L power:GNDD #PWR029
-U 1 1 61EBD066
-P 9400 2450
-F 0 "#PWR029" H 9400 2200 50  0001 C CNN
-F 1 "GNDD" V 9400 2300 50  0000 C CNN
-F 2 "" H 9400 2450 50  0001 C CNN
-F 3 "" H 9400 2450 50  0001 C CNN
-	1    9400 2450
-	0    1    1    0
-$EndComp
-$Comp
 L power:+3.3V #PWR03
 U 1 1 61ECC860
@@
 $EndComp
 $Comp
-L power:+3.3V #PWR030
-U 1 1 61F070E8
-P 9400 2700
-F 0 "#PWR030" H 9400 2550 50  0001 C CNN
-F 1 "+3.3V" V 9400 2950 50  0000 C CNN
-F 2 "" H 9400 2700 50  0001 C CNN
-F 3 "" H 9400 2700 50  0001 C CNN
-	1    9400 2700
-	0    -1   -1   0
-$EndComp
-$Comp
 L power:+5V #PWR025
 U 1 1 61F07825
@@
 	6100 5950 6100 6000
 $Comp
-L Connector:TestPoint TP8
-U 1 1 61FF236E
-P 9400 2700
-F 0 "TP8" V 9350 2900 50  0000 L CNN
-F 1 "+3.3V" V 9450 2600 50  0000 L CNN
-F 2 "TestPoint:TestPoint_THTPad_D1.5mm_Drill0.7mm" H 9600 2700 50  0001 C CNN
-F 3 "~" H 9600 2700 50  0001 C CNN
-	1    9400 2700
-	0    1    1    0
-$EndComp
-$Comp
-L Connector:TestPoint TP9
-U 1 1 61FF42DA
-P 9400 2850
-F 0 "TP9" V 9350 3050 50  0000 L CNN
-F 1 "+5V" V 9450 2750 50  0000 L CNN
-F 2 "TestPoint:TestPoint_THTPad_D1.5mm_Drill0.7mm" H 9600 2850 50  0001 C CNN
-F 3 "~" H 9600 2850 50  0001 C CNN
-	1    9400 2850
-	0    1    1    0
-$EndComp
-$Comp
-L power:+5V #PWR031
-U 1 1 61FF466D
-P 9400 2850
-F 0 "#PWR031" H 9400 2700 50  0001 C CNN
-F 1 "+5V" V 9400 3050 50  0000 C CNN
-F 2 "" H 9400 2850 50  0001 C CNN
-F 3 "" H 9400 2850 50  0001 C CNN
-	1    9400 2850
-	0    -1   -1   0
-$EndComp
-$Comp
 L power:+3.3V #PWR022
