File: rooDialino-KiCad/roodialino.sch (KiCad schematic (older format))
At the start: 50 parts, among them J1 Raspi Connector, J2 ICSP, J3 FTDI, J4 2nd IRX, J5 IR LED, Q1 2N7002, Q2 2N7002, Q3 2N7002, SW1 SW_Push, U1 ATmega328P, U2 TSOP34838, U3 TXS0108EPW, Y1 16 MHz

Commit message: Updating R11 to 0603 footprint in the BOM. JLC won't populate it.
Parts:
- R11: LCSC C25105 -> C23140
Changed lines of the file:
@@
 F 2 "Resistor_SMD:R_0603_1608Metric" V 5330 1300 50  0001 C CNN
 F 3 "~" H 5400 1300 50  0001 C CNN
-F 4 "C25105" H 5400 1300 50  0001 C CNN "LCSC"
+F 4 "C23140" H 5400 1300 50  0001 C CNN "LCSC"
 	1    5400 1300
 	1    0    0    -1
